File: kicad/wireless.kicad_sch (KiCad schematic)
At the start: 4 parts

Commit message: snake, fix pcb errors, update menu
Parts:
- R14: JLCPCB C137872 -> C114877
Changed lines of the file:
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@@
 			)
 		)
-		(property "JLCPCB" "C137872"
+		(property "JLCPCB" "C114877"
 			(at 50.8 43.18 0)
 			(effects
