File: kicad/power.kicad_sch (KiCad schematic)
At the start: 19 parts, among them SW1 EVQPUA02K, U3 TP5400, U6 MAX16054, U7 MCP1825T

Commit message: snake, fix pcb errors, update menu
Parts:
- C1, C29: JLCPCB C77020 -> C49678
Changed lines of the file:
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@@
 			)
 		)
-		(property "JLCPCB" "C77020"
+		(property "JLCPCB" "C49678"
 			(at 57.15 59.69 0)
 			(effects
@@
 			)
 		)
-		(property "JLCPCB" "C77020"
+		(property "JLCPCB" "C49678"
 			(at 137.16 54.61 0)
 			(effects

Commit message: fix bad footprints
Parts:
- L2: JLCPCB C171589 -> C57269
Changed lines of the file:
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@@
 			)
 		)
-		(property "JLCPCB" "C171589"
+		(property "JLCPCB" "C57269"
 			(at 64.77 55.88 0)
 			(effects
