File: kicad/keypad.kicad_sch (KiCad schematic)
At the start: 52 parts, among them Q2 BC847, Q3 BC847, Q4 BC847, Q5 BC847

Commit message: snake, fix pcb errors, update menu
Parts:
- R10, R11, R12, R13, R18, R4, R5, R6: JLCPCB C137872 -> C112291
Changed lines of the file:
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@@
 			)
 		)
-		(property "JLCPCB" "C137872"
+		(property "JLCPCB" "C112291"
 			(at 76.2 161.29 0)
 			(effects
@@
 			)
 		)
-		(property "JLCPCB" "C137872"
+		(property "JLCPCB" "C112291"
 			(at 82.55 104.14 0)
 			(effects
@@
 			)
 		)
-		(property "JLCPCB" "C137872"
+		(property "JLCPCB" "C112291"
 			(at 106.68 26.67 0)
 			(effects
@@
 			)
 		)
-		(property "JLCPCB" "C137872"
+		(property "JLCPCB" "C112291"
 			(at 55.88 26.67 0)
 			(effects
@@
 			)
 		)
-		(property "JLCPCB" "C137872"
+		(property "JLCPCB" "C112291"
 			(at 114.3 26.67 0)
 			(effects
@@
 			)
 		)
-		(property "JLCPCB" "C137872"
+		(property "JLCPCB" "C112291"
 			(at 90.17 104.14 0)
 			(effects
@@
 			)
 		)
-		(property "JLCPCB" "C137872"
+		(property "JLCPCB" "C112291"
 			(at 63.5 26.67 0)
 			(effects
@@
 			)
 		)
-		(property "JLCPCB" "C137872"
+		(property "JLCPCB" "C112291"
 			(at 96.52 161.29 0)
 			(effects

Commit message: remove pull ups
Parts:
- removed R19, R20, R21, R22, R23, R24, R25, R26, R27, R28, R29, R30, R31, R32, R33, R9: 3k, Resistor_SMD:R_0402_1005Metric, symbol Device:R
