File: kicad/brique.kicad_pcb (KiCad board)
At the start: 4 copper layers, 42.1 x 107.7 mm, 126 parts, among them J1 Conn_01x07, J2 USB_B_Micro, J3 Speaker Pads, J4 Battery Connection Pads, J6 BM03B-SRSS-TB, J7 BM03B-SRSS-TB, M1 Vibration, Q1 BC847, Q2 BC847, Q3 BC847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

Commit message: remove flash
Parts:
- removed U1: W25Q128JVS, Package_SO:SOIC-8_5.23x5.23mm_P1.27mm
Routing:
- net QSPI_SCLK: track 14.9 -> 0.00 mm, vias 2 -> 0
- net Net-(U1-IO2): track 19.2 -> 7.34 mm, vias 2 -> 1
- net Net-(U1-DI(IO0)): track 11.4 -> 0.00 mm, vias 2 -> 0
- net Net-(U1-DO(IO1)): track 13.5 -> 2.17 mm, vias 2 -> 1
- net Net-(U1-IO3): track 10.2 -> 5.89 mm, vias 2 -> 1
- net QSPI_SS: track 15.1 -> 11.2 mm

Commit message: update pcb
Parts:
- removed C2: 100nF, Capacitor_SMD:C_0402_1005Metric
- removed R19, R20, R21, R22, R23, R24, R25, R26, R27, R28, R29, R30, R31, R32, R33, R9: 3k, Resistor_SMD:R_0402_1005Metric
Connections:
- net QSPI_SS renamed Net-(U5-QSPI_SS)
- U5 pad 70: Net-(U1-IO3) -> unconnected-(U5-QSPI_SD3-Pad70)
- U5 pad 71: QSPI_SCLK -> unconnected-(U5-QSPI_SCLK-Pad71)
- U5 pad 72: Net-(U1-DI(IO0)) -> unconnected-(U5-QSPI_SD0-Pad72)
- U5 pad 73: Net-(U1-IO2) -> unconnected-(U5-QSPI_SD2-Pad73)
- U5 pad 74: Net-(U1-DO(IO1)) -> unconnected-(U5-QSPI_SD1-Pad74)
Routing:
- net +3V3: track 191.0 -> 124.0 mm, vias 32 -> 30
- net Net-(U1-IO2): track 7.34 -> 0.00 mm, vias 1 -> 0
- net Net-(U1-IO3): track 5.89 -> 0.00 mm, vias 1 -> 0
- net Net-(U1-DO(IO1)): track 2.17 -> 0.00 mm, vias 1 -> 0
- net /Keypad/ZERO: track 96.2 -> 94.6 mm
- net unconnected-(U5-QSPI_SD3-Pad70): track 0.00 -> 1.24 mm
- net /Wireless/DI: track 31.5 -> 30.6 mm
- net /Wireless/~{STANDBY}: track 68.8 -> 68.1 mm
- net Net-(U2-B7_VDDIO): track 11.8 -> 11.1 mm
- net ENABLE: track 16.4 -> 15.8 mm
- net BATTERY+: track 57.8 -> 57.2 mm
- net GND: track 244.7 -> 244.2 mm
- net Net-(JP1-A): track 8.23 -> 7.73 mm

Commit message: update some references for new unavailable chip
Parts:
- U5: value RP2350_80QFN -> RP2354_80QFN
Changed lines of the file:
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@@
 			)
 		)
-		(property "Value" "RP2350_80QFN"
+		(property "Value" "RP2354_80QFN"
 			(at 0 -6.55 270)
 			(layer "B.Fab")
@@
 			)
 		)
-		(property "JLCPCB" "C42415655"
+		(property "JLCPCB" ""
 			(at 0 0 90)
 			(unlocked yes)
